Commit message: Enabling 2D Lidar for husky + Adding supplements box + Enabling move_base to use TEB Local Planner

File: husky_description/urdf/husky.urdf.xacro (robot description, xacro)
@@ -42,5 +42,5 @@
   <xacro:arg name="laser_secondary_rpy"     default="$(optenv HUSKY_LMS1XX_SECONDARY_RPY 0.0 0.0 3.14159)" />
   <!-- UST10 Laser Primary  and Secondary -->
-  <xacro:arg name="laser_ust10_front_enabled" default="$(optenv HUSKY_UST10_ENABLED 0)" />
+  <xacro:arg name="laser_ust10_front_enabled" default="$(optenv HUSKY_UST10_ENABLED 1)" />
   <xacro:arg name="laser_ust10_front_topic"   default="$(optenv HUSKY_UST10_TOPIC front/scan)" />
   <xacro:arg name="laser_ust10_front_prefix"  default="$(optenv HUSKY_UST10_PREFIX front)" />
@@ -155,4 +155,35 @@
     </collision>
   </link>
+  <!-- Supplements Box Object -->
+  <joint name="supplements_box" type="fixed">
+    <parent link="base_link"/>
+    <child link="obj_box"/>
+  </joint>
+  <link name="obj_box">
+    <collision>
+      <origin xyz="-0.04 0 ${base_z_size+0.2}" rpy="0 0 0"/>
+      <geometry>
+	       <box size="${base_x_size*0.5} ${base_y_size*0.8} ${base_z_size*1.5}"/>
+      </geometry>
+    </collision>
+    <visual>
+      <origin xyz="-0.04 0 ${base_z_size+0.2}" rpy="0 0 0"/>
+      <geometry>
+	       <box size="${base_x_size*0.5} ${base_y_size*0.8} ${base_z_size*1.5}"/>
+      </geometry>
+      <material name="red"/>
+    </visual>
+    <inertial>
+      <origin xyz="-0.04 0 ${base_z_size+0.2}" rpy="0 0 0"/>
+      <mass value="10"/>
+      <inertia
+    	  ixx="1.0" ixy="0.0" ixz="0.0"
+    	  iyy="1.0" iyz="0.0"
+    	  izz="1.0"/>
+    </inertial>
+  </link>
+  <gazebo reference="obj_box">
+    <material>Gazebo/Red</material>
+  </gazebo>
   <!-- Base footprint is on the ground under the robot -->
   <link name="base_footprint"/>
